File: Jetson_Extension_Board2.5.1.kicad_pcb (KiCad board)
At the start: 2 copper layers, 18 parts, among them J10 TBP03R2-350-03BE, J2 TBP03R2-350-03BE, J3 TBP03R2-350-03BE, J4 TBP03R2-350-03BE, J5 TBP03R2-350-03BE, J6 40_Pin_Jetson_Connector, J7 TBP03R2-350-03BE, J8 TBP03R2-350-03BE, J9 TBP03R2-350-03BE, U1 BNO055, U2 74LV14, U4 ADS1115IDGS

Commit message: PCB Layout attempted 1
Parts:
- moved J10 20.7 mm to (149.5, 122.0)
- moved J3 13.9 mm to (155.5, 155.0)
- moved J7 9.91 mm to (129.5, 108.0)
- moved J8 9.41 mm to (129.5, 116.2)
- moved J9 9.41 mm to (129.5, 125.0)
- moved U4 9.01 mm to (132.3, 99.0)
- moved J5 8.56 mm to (121.8, 154.0)
- moved R2 6.61 mm to (146.0, 109.2)
- moved U1 6.61 mm to (152.2, 105.8)
- moved C1 6.61 mm to (146.0, 104.2)
- moved C2 6.61 mm to (149.5, 99.2)
- moved C3 6.61 mm to (154.5, 99.2)
- moved C4 6.61 mm to (152.5, 112.7)
- moved R1 6.61 mm to (158.5, 105.6)
- moved J2 5.31 mm to (154.5, 130.5), turned to -90 degrees
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