File: Jetson_Extension_Board(Pluh2).kicad_pcb (KiCad board)
At the start: 2 copper layers, 25 parts, among them J1 I2C_2 DEBUG, J10 TBP03R2-350-03BE, J11 ST DEBUG, J2 TBP03R2-350-03BE, J3 TBP03R2-350-03BE, J4 TBP03R2-350-03BE, J5 TBP03R2-350-03BE, J6 40_Pin_Jetson_Connector, J7 TBP03R2-350-03BE, J8 TBP03R2-350-03BE, J9 TBP03R2-350-03BE, SW1 SW_Push_DPDT, U1 BNO055, U2 74LV14, U4 ADS1115IDGS

Commit message: Freerouted attempt
Routing:
- net GND: track 0.00 -> 317.5 mm
- net /ADC/3.3V: track 0.00 -> 191.8 mm
- net /I2C_2_SDA: track 0.00 -> 138.9 mm, vias 0 -> 1
- net /SchmittTrigger(74LV14)/5V: track 0.00 -> 109.4 mm
- net /I2C_2_SCL: track 0.00 -> 93.2 mm, vias 0 -> 2
- net ADC ALERT: track 0.00 -> 82.1 mm, vias 0 -> 1
- net ST 1: track 0.00 -> 64.1 mm
- net IMU nBOOT: track 0.00 -> 62.2 mm, vias 0 -> 1
- net IMU INT: track 0.00 -> 55.5 mm
- net ST 2: track 0.00 -> 54.2 mm
- net IMU nRESET: track 0.00 -> 52.9 mm, vias 0 -> 1
- net COM 3: track 0.00 -> 51.5 mm
- net ST 3: track 0.00 -> 46.8 mm
- net 3.3V: track 0.00 -> 46.7 mm
- net /ADC/Signal 1: track 0.00 -> 44.6 mm
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Other:
- board outline added: 94.5 x 79.5 mm
- board text added: "Jetson Extension Board 10/27/2024 Rev. 2"

Commit message: More stuff yuh
Parts:
- added G***: LOGO, LOGO, F.Cu at (155.5, 109.0)
Other:
- board text added: "3.3V"
- board text added: "5V"
- board text added: "ADC INPUTS"
- board text added: "C1"
- board text added: "C6"
- board text added: "C7"
- board text added: "C8"
- board text added: "GND"
- board text added: "J1"
- board text added: "J10"
- board text added: "J11"
- board text added: "J2"
- board text added: "J3"
- board text added: "J4"
- board text added: "J7"
- board text added: "J8"
- board text added: "J9"
- board text added: "R1"
- board text added: "R2"
- board text added: "SCHMITT TRIGGER INPUTS"
- board text added: "Sig 1"
- board text added: "Sig 2"
- board text added: "Sig 3"
- board text added: "Sig 4"
- board text added: "U1"
- board text added: "U2"
- board text added: "U4"
