File: ADC.kicad_sch (KiCad schematic)
At the start: 6 parts, among them J1 I2C_2 DEBUG, J10 TBP03R2-350-03BE, J7 TBP03R2-350-03BE, J8 TBP03R2-350-03BE, J9 TBP03R2-350-03BE, U4 ADS1115IDGS

Commit message: PCB Update
Parts:
- added C2: 0.1u, Capacitor_SMD:C_1206_3216Metric, symbol Device:C
Connections:
- net 3.3V: now also C2.1
- net GND: now also C2.2
Changed lines of the file:
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@@
+	)
+	(junction
+		(at 149.86 52.07)
+		(diameter 0)
+		(color 0 0 0 0)
 	)
 	(junction
@@
 	(wire
 		(pts
+			(xy 195.58 71.12) (xy 195.58 87.63)
+		)
+		(stroke
+			(width 0)
+			(type default)
+		)
+	)
+	(wire
+		(pts
 			(xy 135.89 62.23) (xy 106.68 62.23)
 		)
@@
 	(wire
 		(pts
+			(xy 195.58 48.26) (xy 158.75 48.26)
+		)
+		(stroke
+			(width 0)
+			(type default)
+		)
+	)
+	(wire
+		(pts
+			(xy 149.86 52.07) (xy 149.86 60.96)
+		)
+		(stroke
+			(width 0)
+			(type default)
+			(color 255 0 0 1)
+		)
+	)
+	(wire
+		(pts
 			(xy 166.37 80.01) (xy 170.18 80.01)
 		)
@@
 	(wire
 		(pts
+			(xy 158.75 48.26) (xy 158.75 52.07)
+		)
+		(stroke
+			(width 0)
+			(type default)
+		)
+	)
+	(wire
+		(pts
 			(xy 149.86 83.82) (xy 149.86 87.63)
 		)
@@
 	(wire
 		(pts
-			(xy 149.86 48.26) (xy 149.86 60.96)
-		)
-		(stroke
-			(width 0)
-			(type default)
-			(color 255 0 0 1)
+			(xy 149.86 48.26) (xy 149.86 52.07)
+		)
+		(stroke
+			(width 0)
+			(type default)
+			(color 255 0 0 1)
+		)
+	)
+	(wire
+		(pts
+			(xy 195.58 48.26) (xy 195.58 63.5)
+		)
+		(stroke
+			(width 0)
+			(type default)
 		)
 	)
@@
 			(type solid)
 			(color 1 0 0 1)
+		)
+	)
+	(wire
+		(pts
+			(xy 158.75 52.07) (xy 149.86 52.07)
+		)
+		(stroke
+			(width 0)
+			(type default)
+		)
+	)
+	(wire
+		(pts
+			(xy 195.58 87.63) (xy 149.86 87.63)
+		)
+		(stroke
+			(width 0)
+			(type default)
 		)
 	)
@@
 					(unit 1)
 				)
+			)
+		)
+	)
+	(symbol
+		(lib_id "Device:C")
+		(at 195.58 67.31 0)
+		(unit 1)
+		(exclude_from_sim no)
+		(in_bom yes)
+		(on_board yes)
+		(dnp no)
+		(fields_autoplaced yes)
+		(property "Reference" "C2"
+			(at 199.39 66.0399 0)
+			(effects
+				(font
+					(size 1.27 1.27)
+				)
+				(justify left)
+			)
+		)
+		(property "Value" "0.1u"
+			(at 199.39 68.5799 0)
+			(effects
+				(font
+					(size 1.27 1.27)
+				)
+				(justify left)
+			)
+		)
+		(property "Footprint" "Capacitor_SMD:C_1206_3216Metric"
+			(at 196.5452 71.12 0)
+			(effects
+				(font
+					(size 1.27 1.27)
+				)
+				(hide yes)
+			)
+		)
+		(property "Datasheet" "~"
+			(at 195.58 67.31 0)
+			(effects
+				(font
+					(size 1.27 1.27)
+				)
+				(hide yes)
+			)
+		)
+		(property "Description" "Unpolarized capacitor"
+			(at 195.58 67.31 0)
+			(effects
+				(font
+					(size 1.27 1.27)
+				)
+				(hide yes)
+			)
+		)
+		(pin "1"
+		)
+		(pin "2"
+		)
+		(instances
+			(project "Jetson_Extension_Board"
+				(path "/fac81d63-8655-47f4-bf8e-62708c29b8c6/607cc1b6-24e0-474a-81e8-dcba676951e3"
+					(reference "C2")
+					(unit 1)
+				)
